File: MD_CAN_Tester.kicad_pcb (KiCad board)
At the start: 2 copper layers, 35 parts, among them J1 USB_B_Micro, J2 SWD, J3 AnalogInput, J4 PinHeader, J5 CAN_Connector, SW1 USER_BUTTON, SW2 ID_SELECT, U1 STM32F446RETx, U2 MCP1703A-3002_SOT223, U3 MCP2562-E-SN

Commit message: GND以外ほぼ配線済み
Parts:
- removed J2: SWD, LibLoader:FTSH-107-XX-YYY-DV-K-A-TR
- removed JP1: TXD_EN, Connector_PinHeader_2.54mm:PinHeader_1x02_P2.54mm_Vertical
- removed JP2: Rteam_EN, Connector_PinHeader_2.54mm:PinHeader_1x02_P2.54mm_Vertical
- added C6: 0.1u, Capacitor_SMD:C_0603_1608Metric, F.Cu at (-6.75, 0.68)
- added C7: 0.1u, Capacitor_SMD:C_0603_1608Metric, F.Cu at (-1.09, 13.5)
- added C8: 0.1u, Capacitor_SMD:C_0603_1608Metric, F.Cu at (1.39, -3.92)
- added C9: 0.1u, Capacitor_SMD:C_0603_1608Metric, F.Cu at (9.00, 6.00)
- added R11: 0R, Resistor_SMD:R_0603_1608Metric, F.Cu at (-6.50, 20.5)
- added R12: 0R, Resistor_SMD:R_0603_1608Metric, F.Cu at (-2.50, 17.5)
- added R_term: Rteam_EN, Connector_PinHeader_2.54mm:PinHeader_1x02_P2.54mm_Vertical, F.Cu at (10.0, -19.0)
- added SWD: SWD, LibLoader:FTSH-107-XX-YYY-DV-K-A-TR, F.Cu at (-13.5, 6.50)
- added TXD_EN: TXD_EN, Connector_PinHeader_2.54mm:PinHeader_1x02_P2.54mm_Vertical, F.Cu at (-12.5, -3.50)
- U2: value MCP1703A-3002_SOT223 -> MCP1703A-3302_SOT23; footprint Package_TO_SOT_SMD:SOT-223-3_TabPin2 -> LibLoader:SOT95P255X145-3N
- moved R7 179.7 mm to (-15.5, -16.5), turned to 270 degrees
- moved C5 169.9 mm to (-13.5, -6.50), turned to 180 degrees
- moved C4 167.8 mm to (-10.0, -11.0), turned to 270 degrees
- moved 5V 167.5 mm to (-4.00, -22.0)
- moved H 165.4 mm to (0.00, -22.0)
- moved R6 165.0 mm to (-9.50, -2.50), turned to 90 degrees
- moved L 162.9 mm to (4.00, -22.0)
- moved 5V_EN 162.7 mm to (-10.0, -19.0), turned to 180 degrees
- moved R10 162.0 mm to (7.00, -18.5), turned to 270 degrees
- moved R8 159.4 mm to (0.00, -8.00), turned to 180 degrees
- moved U3 158.7 mm to (-13.5, -11.0), turned to 90 degrees
- moved R2 158.6 mm to (-3.92, -2.15), turned to 225 degrees
- moved R4 155.8 mm to (10.5, -9.50), turned to 90 degrees
- moved C1 153.0 mm to (-3.21, 12.0), turned to 315 degrees
- moved R5 152.3 mm to (10.5, -5.50), turned to 90 degrees
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- renumbered TP3 to 5V, JP3 to 5V_EN, TP4 to GND, TP1 to H, TP2 to L
Connections:
- J1 pad 4: GND -> Net-(J1-Pad4)
- J1 pad 6: GND -> Net-(J1-Pad6)
- U1 pad 10: Net-(U1-Pad10) -> (no net)
- U1 pad 11: Net-(U1-Pad11) -> (no net)
- U1 pad 15: Net-(U1-Pad15) -> (no net)
- U1 pad 2: Net-(U1-Pad2) -> (no net)
- U1 pad 20: Net-(U1-Pad20) -> (no net)
- U1 pad 21: Net-(U1-Pad21) -> (no net)
- U1 pad 22: Net-(U1-Pad22) -> (no net)
- U1 pad 23: Net-(U1-Pad23) -> (no net)
- U1 pad 24: Net-(U1-Pad24) -> (no net)
- U1 pad 25: Net-(U1-Pad25) -> (no net)
- U1 pad 27: Net-(U1-Pad27) -> (no net)
- U1 pad 28: Net-(U1-Pad28) -> (no net)
- U1 pad 3: Net-(U1-Pad3) -> (no net)
- U1 pad 37: Net-(U1-Pad37) -> (no net)
- U1 pad 38: Net-(U1-Pad38) -> (no net)
- U1 pad 39: Net-(U1-Pad39) -> (no net)
- U1 pad 4: Net-(U1-Pad4) -> (no net)
- U1 pad 40: Net-(U1-Pad40) -> (no net)
- U1 pad 41: Net-(U1-Pad41) -> (no net)
- U1 pad 43: Net-(U1-Pad43) -> (no net)
- U1 pad 5: Net-(U1-Pad5) -> (no net)
- U1 pad 50: Net-(U1-Pad50) -> (no net)
- U1 pad 51: Net-(U1-Pad51) -> (no net)
- U1 pad 52: Net-(U1-Pad52) -> (no net)
- U1 pad 53: Net-(U1-Pad53) -> (no net)
- U1 pad 54: Net-(U1-Pad54) -> (no net)
- U1 pad 56: Net-(U1-Pad56) -> (no net)
- U1 pad 57: Net-(U1-Pad57) -> (no net)
- U1 pad 58: Net-(U1-Pad58) -> (no net)
- U1 pad 59: Net-(U1-Pad59) -> (no net)
- U1 pad 6: Net-(U1-Pad6) -> (no net)
- U1 pad 8: Net-(U1-Pad8) -> (no net)
- U1 pad 9: Net-(U1-Pad9) -> (no net)
- U2 pad 1: +5V -> GND
- U2 pad 2: GND -> +3V3
- U2 pad 3: +3V3 -> +5V
Routing:
- net +3V3: track 0.00 -> 138.5 mm
- net +5V: track 0.00 -> 76.0 mm, vias 0 -> 3
- net GND: track 0.00 -> 44.7 mm
- net Net-(J4-Pad4): track 0.00 -> 44.7 mm
- net Net-(J4-Pad3): track 0.00 -> 42.4 mm, vias 0 -> 2
- net Net-(R8-Pad2): track 0.00 -> 33.3 mm, vias 0 -> 2
- net Net-(J3-Pad2): track 0.00 -> 30.8 mm, vias 0 -> 2
- net T_SWDIO: track 0.00 -> 24.9 mm, vias 0 -> 2
- net T_SWCLK: track 0.00 -> 24.8 mm, vias 0 -> 2
- net T_SWO: track 0.00 -> 22.3 mm, vias 0 -> 2
- net /CAN1_TX: track 0.00 -> 21.0 mm, vias 0 -> 1
- net Net-(J4-Pad1): track 0.00 -> 20.0 mm
- net /CAN1_RX: track 0.00 -> 19.5 mm, vias 0 -> 2
- net T_VCP_TX: track 0.00 -> 18.9 mm, vias 0 -> 2
- net /USB_DP: track 0.00 -> 17.9 mm, vias 0 -> 2
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Other:
- board outline added: 36 x 47.5 mm
- board text added: "5V"
- board text added: "CANH"
- board text added: "CANL"
- board text added: "GND"

Commit message: 配線完了
Parts:
- moved SWD 2.25 mm to (-13.5, 8.75)
- moved R12 0.90 mm to (-3.25, 17.0)
Routing:
- net GND: track 44.7 -> 233.7 mm, vias 0 -> 70
- net +5V: track 76.0 -> 67.0 mm, vias 3 -> 5
- net T_SWCLK: track 24.8 -> 27.8 mm
- net Net-(R8-Pad2): track 33.3 -> 35.3 mm
- net +3V3: track 138.5 -> 140.0 mm
- net T_VCP_TX: track 18.9 -> 17.5 mm
- net Net-(J1-Pad4): track 2.51 -> 3.80 mm
- net Net-(J4-Pad4): track 44.7 -> 43.6 mm
- net Net-(J4-Pad3): track 42.4 -> 41.3 mm
- net Net-(J3-Pad2): track 30.8 -> 31.8 mm
- net T_VCP_RX: track 8.53 -> 7.59 mm
- net T_SWO: track 22.3 -> 23.2 mm
- net T_NRST: track 16.1 -> 17.0 mm
- net Net-(SW1-Pad1): track 17.0 -> 17.8 mm
- net /USB_DM: track 16.1 -> 16.8 mm
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- added copper zone on B.Cu, net GND
- added copper zone on F.Cu, net GND
Other:
- net class Default: clearance 0.2 -> 0.11
- rule trace_clearance: 0.2 -> 0.11
- rule trace_min: 0.2 -> 0.11
- board text added: "CAN Tester ver.1 Designed by @akito_0914."
